File: modules/OBJEX_M0-HDC1080/OBJEX_M0-HDC1080.sch (KiCad schematic (older format))
At the start: 6 parts, among them J1 BM28B0.6-16DP_2-0.35V(51), J3 BM28B0.6-16DP_2-0.35V(51), U1 HDC1080

Commit message: update
Parts:
- added D2: 1N4148WS, Diode_SMD:D_SOD-323, symbol Device:D
- C1: footprint Capacitor_SMD:C_0603_1608Metric -> Capacitor_SMD:C_0402_1005Metric
Connections:
- net labels added: VCC
- wire segments 35 -> 36
Other:
- note removed: "CAUTION: NO REVERSE POLARITY/ESD PROTECTION!"
- note removed: "M0 - HDC1080 v1.0"
- moved on the sheet: C1, J1, J3, R1, R2, U1
