File: modules/OBJEX_M0-HDC1080/OBJEX_M0-HDC1080.kicad_pcb (KiCad board)
At the start: 2 copper layers, 20.1 x 10 mm, 7 parts, among them J1 BM28B0.6-16DP_2-0.35V(51), J3 BM28B0.6-16DP_2-0.35V(51), U1 HDC1080

Commit message: update
Parts:
- removed the G*** at (144.0, 90.2)
- added D2: D, Diode_SMD:D_SOD-323, F.Cu at (150.7, 90.9)
- added G***: LOGO, KicadLibrary:arrowTiny, F.Cu at (144.0, 93.7)
- added G***: LOGO, KicadLibrary:logov2-mini, B.Cu at (144.0, 90.2)
- C1: footprint Capacitor_SMD:C_0603_1608Metric -> Capacitor_SMD:C_0402_1005Metric
- moved C1 0.77 mm to (148.2, 90.8)
Connections:
- C1 pad 2: +3V3 -> VCC
- R1 pad 1: +3V3 -> VCC
- R2 pad 1: +3V3 -> VCC
- U1 pad 5: +3V3 -> VCC
Routing:
- net VCC: track 0.00 -> 15.6 mm
- net +3V3: track 17.2 -> 3.48 mm, vias 2 -> 1
- net Net-(J1-Pad10): track 1.32 -> 0.00 mm, vias 1 -> 0
- net Net-(J1-Pad14): track 1.31 -> 0.00 mm, vias 1 -> 0
- net Net-(J1-Pad15): track 0.00 -> 0.90 mm, vias 0 -> 1
- net Net-(J1-Pad11): track 0.00 -> 0.89 mm, vias 0 -> 1
- net Net-(U1-Pad7): vias 0 -> 6
- net GND: vias 5 -> 2
- removed copper zone on B.Cu, net GND
Other:
- board text removed: "Copyright CERN 2020. This source describes Open Hardware and is licensed under the CERN-OHLW v2 You may redistribute and modify this documentation and make products using it under the terms of the CERN-OHL-W v2 (https:/cern.ch/cern-ohl). This documentation is distributed WITHOUT ANY EXPRESS OR IMPLIED WARRANTY, INCLUDING OF MERCHANTABILITY, SATISFACTORY QUALITY AND FITNESS FOR A PARTICULAR PURPOS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"

Commit message: Update KiCad 6.0.0
Other:
- net class Default removed
