File: modules/OBJEX_M1-BTN/OBJEX_M1-BTN.sch (KiCad schematic (older format))
At the start: 14 parts, among them J1 BM28B0.6-16DP_2-0.35V(51), J2 BM28B0.6-16DP_2-0.35V(51), J3 BM28B0.6-16DP_2-0.35V(51), J4 BM28B0.6-16DP_2-0.35V(51), SW1 SW_Push

Commit message: update rev1.5
Parts:
- removed D1, D2, D3, D4: LED, LED_SMD:LED_0603_1608Metric, symbol Device:LED
- removed R2, R3, R4, R5: 220, Resistor_SMD:R_0603_1608Metric, symbol Device:R
- added C1, C2, C3, C4: 0.1uF, Capacitor_SMD:C_0402_1005Metric, symbol Device:C
- added D1: 1N4148WS, Diode_SMD:D_SOD-323, symbol Device:D
- added U1, U2, U3, U4: WS2812-2020, KicadLibrary:LED_WS2812-2020, symbol WS2812-2020:WS2812-2020
- added U5: TJE-533-S-V-T_R, Button_Switch_SMD:TJE-533, symbol Switch:TJE-533-S-V-T_R
- R1: footprint Resistor_SMD:R_0603_1608Metric -> Resistor_SMD:R_0402_1005Metric
Connections:
- net labels added: RGB-OUT, VCC
- wire segments 66 -> 92
Other:
- note removed: "CAUTION: NO REVERSE POLARITY/ESD PROTECTION!"
- note removed: "M1 - BTN v1.0"
- note removed: "Socket\nOBJEX LINK rev1.0"
- moved on the sheet: J1, J2, J3, J4, R1, SW1
