File: modules/OBJEX_M1-BTN/OBJEX_M1-BTN.kicad_pcb (KiCad board)
At the start: 2 copper layers, 20.1 x 20.2 mm, 15 parts, among them J1 BM28B0.6-16DP_2-0.35V(51), J2 BM28B0.6-16DP_2-0.35V(51), J3 BM28B0.6-16DP_2-0.35V(51), J4 BM28B0.6-16DP_2-0.35V(51), SW1 SW_Push

Commit message: update rev1.5
Parts:
- removed D2, D3, D4: LED, LED_SMD:LED_0603_1608Metric
- removed the G*** at (144.0, 95.2)
- removed R2, R3, R4, R5: 220, Resistor_SMD:R_0603_1608Metric
- added C1: 0.1uF, Capacitor_SMD:C_0402_1005Metric, F.Cu at (135.1, 97.7)
- added C2: 0.1uF, Capacitor_SMD:C_0402_1005Metric, F.Cu at (153.1, 92.9)
- added C3: 0.1uF, Capacitor_SMD:C_0402_1005Metric, F.Cu at (141.4, 104.3)
- added C4: 0.1uF, Capacitor_SMD:C_0402_1005Metric, F.Cu at (146.7, 86.6)
- added G***: LOGO, KicadLibrary:arrowTiny, F.Cu at (150.8, 103.5)
- added G***: LOGO, KicadLibrary:logov2-mini, B.Cu at (143.9, 95.3)
- added U1: WS2812-2020, KicadLibrary:LED_WS2812-2020, F.Cu at (144.0, 103.5)
- added U2: WS2812-2020, KicadLibrary:LED_WS2812-2020, F.Cu at (144.0, 87.1)
- added U3: WS2812-2020, KicadLibrary:LED_WS2812-2020, F.Cu at (152.0, 95.3)
- added U4: WS2812-2020, KicadLibrary:LED_WS2812-2020, F.Cu at (136.1, 95.2)
- added U5: TJE-533-S-V-T_R, Button_Switch_SMD:TJE-533, F.Cu at (144.0, 90.5)
- D1: value LED -> 1N4148WS; footprint LED_SMD:LED_0603_1608Metric -> Diode_SMD:D_SOD-323
- R1: value 1K -> 10K; footprint Resistor_SMD:R_0603_1608Metric -> Resistor_SMD:R_0402_1005Metric
- moved D1 18.8 mm to (152.8, 89.7)
- moved R1 4.25 mm to (151.1, 100.5)
Connections:
- D1 pad 1: GND -> +3V3
- J1 pad 19: +3V3 -> Net-(D1-Pad2)
- J1 pad 20: +3V3 -> Net-(D1-Pad2)
- J2 pad 19: +3V3 -> Net-(D1-Pad2)
- J2 pad 20: +3V3 -> Net-(D1-Pad2)
- J4 pad 19: +5V -> VCC
- J4 pad 20: +5V -> VCC
- J4 pad 8: Net-(J4-Pad8) -> RGB-OUT
Routing:
- net +3V3: track 7.71 -> 50.6 mm, vias 2 -> 0
- net Net-(U1-Pad1): track 0.00 -> 15.5 mm
- net IO26: track 15.0 -> 0.00 mm, vias 1 -> 0
- net Net-(U2-Pad1): track 0.00 -> 13.8 mm
- net IO25: track 11.5 -> 0.00 mm, vias 1 -> 0
- net Net-(U2-Pad3): track 0.00 -> 10.9 mm, vias 0 -> 2
- net Net-(D1-Pad2): track 1.57 -> 11.6 mm, vias 0 -> 2
- net IO27: track 6.34 -> 0.00 mm, vias 1 -> 0
- net RGB-OUT: track 0.00 -> 5.83 mm, vias 0 -> 1
- net Net-(J1-Pad6): track 5.04 -> 0.00 mm, vias 1 -> 0
- net IO23: track 3.97 -> 0.00 mm, vias 1 -> 0
- net VCC: track 0.00 -> 2.83 mm, vias 0 -> 1
- net +5V: track 6.31 -> 3.48 mm, vias 2 -> 1
- net GND: track 18.4 -> 20.9 mm, vias 9 -> 14
- net Net-(J4-Pad15): track 1.90 -> 0.00 mm, vias 1 -> 0
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Other:
- board text added: "IoT BTN"
- board text removed: "BTN"
- board text removed: "Copyright CERN 2020. This source describes Open Hardware and is licensed under the CERN-OHLW v2 You may redistribute and modify this documentation and make products using it under the terms of the CERN-OHL-W v2 (https:/cern.ch/cern-ohl). This documentation is distributed WITHOUT ANY EXPRESS OR IMPLIED WARRANTY, INCLUDING OF MERCHANTABILITY, SATISFACTORY QUALITY AND FITNESS FOR A PARTICULAR PURPOS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"

Commit message: Update KiCad 6.0.0
Other:
- net class Default removed
