File: modules/OBJEX_M0-LIS3DHTR.VL53L0X/OBJEX_M0-LIS3DHTR.VL53L0X.kicad_pcb (KiCad board)
At the start: 2 copper layers, 20.1 x 10 mm, 16 parts, among them J1 BM28B0.6-16DP_2-0.35V(51), J3 BM28B0.6-16DP_2-0.35V(51), U1 LIS3DH, U2 VL53L0X

Commit message: Update KiCad 6.0.0
Other:
- net class Default removed
