File: modules/OBJEX_M0-MPU6050/OBJEX_M0-MPU6050.kicad_pcb (KiCad board)
At the start: 2 copper layers, 20.1 x 10 mm, 11 parts, among them J1 BM28B0.6-16DP_2-0.35V(51), J3 BM28B0.6-16DP_2-0.35V(51), U1 MPU6050

Commit message: Update KiCad 6.0.0
Other:
- net class Default removed
