File: modules/OBJEX_M0-PSRAM_LY68L6400SLIT/PSRAM_LY68L6400SLIT.kicad_pcb (KiCad board)
At the start: 2 copper layers, 20.1 x 10 mm, 7 parts, among them J1 BM28B0.6-16DP_2-0.35V(51), J3 BM28B0.6-16DP_2-0.35V(51), U1 ESP-PSRAM32

Commit message: Update KiCad 6.0.0
Other:
- net class Default removed
