File: modules/OBJEX_Socket-V2.0/OBJEX_Socket-V2.0.kicad_pcb (KiCad board)
At the start: 2 copper layers, 20.1 x 20.2 mm, 7 parts, among them J1 BM28B0.6-16DP_2-0.35V(51), J2 BM28B0.6-16DP_2-0.35V(51), J3 BM28B0.6-16DP_2-0.35V(51), J4 BM28B0.6-16DP_2-0.35V(51), U1 OBJEX_SOCKET_V2

Commit message: Update KiCad 6.0.0
Other:
- net class Default removed
