File: modules/ProtoBoard_v2.0/ProtoBoard_v2.0.kicad_pcb (KiCad board)
At the start: 2 copper layers, 62.5 x 26.7 mm, 29 parts, among them J1 Conn_01x10, J2 Conn_01x10, J3 Conn_01x10, J4 Conn_01x10, U1 OBJEX_SOCKET_V2-pads

Commit message: Update KiCad 6.0.0
Other:
- net class Default removed
